File: dobrock69-parts.kicad_pcb (KiCad board)
At the start: 2 copper layers, 85.4 x 83 mm, 34 parts

Commit message: Dobrock69 kansei!
Parts:
- removed the REF** at (191.6, 112.7)
- added MX1: MX-NoLED, miyajima:MXOnly-1U-Hotswap-0.8mm-parts, F.Cu at (191.4, 112.7)
Other:
- outline, holes or cut-outs redrawn
- board text added: "Bottom Side"
- board text added: "Front Side"
