File: dobrock69.kicad_pcb (KiCad board)
At the start: 2 copper layers, 159 parts, among them J1 HDMI_A_1.4, J2 Conn_01x02, J3 Conn_01x03, U1 XC6206P332MR, U2 STM32L072KBUx

Commit message: PCB switch daitai haichi shita
Parts:
- MX59, MX60, MX61, MX64, MX65, MX66: footprint kbd:CherryMX_Choc_Hotswap -> kbd:Choc_Hotswap
- moved C2 437.3 mm to (448.8, 235.5)
- moved D12 313.7 mm to (551.9, 142.0)
- moved D27 313.7 mm to (563.9, 128.9)
- moved D6 313.7 mm to (551.9, 144.9)
- moved D9 313.7 mm to (563.9, 131.8)
- moved R2 313.7 mm to (592.2, 87.2)
- moved R3 313.7 mm to (592.2, 89.7)
- moved C1 313.7 mm to (439.0, 88.0)
- moved C3 313.7 mm to (406.7, 214.3)
- moved C4 313.7 mm to (357.1, 150.8)
- moved C5 313.7 mm to (433.2, 88.0)
- moved C6 313.7 mm to (436.1, 88.0)
- moved C7 313.7 mm to (421.9, 108.8)
- moved D1 313.7 mm to (547.5, 147.9)
- moved D10 313.7 mm to (502.9, 192.4)
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
Commit message: pcb susunda
Parts:
- D60, D61, D63, D65, D69, J1: moved to B.Cu
- MX1, MX10, MX11, MX12, MX13, MX14, MX15, MX16, MX18, MX19, MX20, MX21, MX22, MX23, MX24, MX25, MX26, MX27, MX28, MX3, MX30, MX32, MX33, MX34, MX35, MX36, MX37, MX38, MX39, MX4, MX40, MX41, MX42, MX44, MX45, MX49, MX5, MX50, MX53, MX54, MX55, MX56, MX57, MX58, MX6, MX62, MX63, MX67, MX68, MX69, MX7, MX8, MX9: footprint MX_Only:MXOnly-1U-Hotswap -> MX_Only:MXOnly-1U-NoLED
- MX17, MX29: footprint MX_Only:MXOnly-1.75U-Hotswap -> MX_Only:MXOnly-1.75U-NoLED
- MX2: footprint MX_Only:MXOnly-1.5U-Hotswap -> MX_Only:MXOnly-1.5U-NoLED
- MX31, MX43, MX48, MX51: footprint MX_Only:MXOnly-2.25U-Hotswap -> MX_Only:MXOnly-2.25U-NoLED
- MX46, MX47, MX52: footprint MX_Only:MXOnly-1.25U-Hotswap -> MX_Only:MXOnly-1.25U-NoLED
- MX59, MX60, MX61, MX64, MX65, MX66: footprint kbd:Choc_Hotswap -> Kailh_Choc:KailhChoc-1U
- moved J1 404.1 mm to (183.1, 28.4), turned to 270 degrees
- moved MX23 104.7 mm to (41.6, 222.7)
- moved MX37 104.7 mm to (37.4, 243.6)
- moved MX8 104.7 mm to (32.1, 205.5)
- moved MX24 104.7 mm to (60.0, 217.8)
- moved MX38 104.7 mm to (55.8, 238.6)
- moved MX9 104.7 mm to (50.5, 200.6)
- moved MX10 104.7 mm to (68.9, 195.7)
- moved MX25 104.7 mm to (78.5, 212.8)
- moved MX39 104.7 mm to (74.2, 233.7)
- moved MX51 104.7 mm to (66.8, 255.8)
- moved MX52 104.7 mm to (99.1, 247.7)
- moved MX63 104.7 mm to (54.9, 279.3)
- moved MX64 104.7 mm to (73.3, 274.4)
- moved MX65 104.7 mm to (91.7, 269.5)
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Other:
- board outline added: 180 x 277.4 mm

Commit message: pcb haisen susunda
Parts:
- C1, C2, C3, C4, C5, C6, C7, D1, D10, D11, D12, D13, D14, D15, D16, D17, D18, D19, D2, D20, D21, D22, D23, D24, D25, D26, D27, D28, D29, D3, D30, D31, D32, D33, D34, D35, D36, D37, D38, D39, D4, D40, D41, D42, D43, D44, D45, D46, D47, D48, D49, D5, D50, D51, D52, D53, D54, D55, D56, D57, D58, D59, D6, D62, D64, D66, D67, D68, D7, D8, D9, ESD1, ESD2, F1, J2, J3, R1, R2, R3, SW_BOOT1, SW_RESET1, U1, U2: moved to B.Cu
- J1: moved to F.Cu
- MX31, MX43, MX48, MX51: footprint MX_Only:MXOnly-2.25U-NoLED -> MX_Only:MXOnly-2.25U-ReversedStabilizers-NoLED
- moved D1 509.9 mm to (51.3, 30.3), turned to 90 degrees
- moved D16 501.3 mm to (48.1, 48.5), turned to 90 degrees
- moved D46 501.2 mm to (88.6, 87.1), turned to 90 degrees
- moved D17 499.6 mm to (53.7, 48.5), turned to 90 degrees
- moved D47 493.8 mm to (96.1, 87.4), turned to 90 degrees
- moved D2 490.5 mm to (56.9, 30.2), turned to 90 degrees
- moved D5 465.8 mm to (122.7, 33.0), turned to 90 degrees
- moved D3 465.7 mm to (79.9, 29.5), turned to 90 degrees
- moved D18 460.8 mm to (78.3, 48.5), turned to 90 degrees
- moved D4 457.8 mm to (102.1, 29.8), turned to 90 degrees
- moved D31 449.2 mm to (46.5, 68.4), turned to 90 degrees
- moved D32 446.5 mm to (83.1, 67.9), turned to 90 degrees
- moved D33 438.9 mm to (106.5, 68.4), turned to 90 degrees
- moved D44 434.6 mm to (45.7, 87.4), turned to 90 degrees
- moved D6 424.6 mm to (141.0, 38.2), turned to 90 degrees
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Routing:
- net ROW3: track 0.00 -> 495.5 mm, vias 0 -> 1
- net ROW4: track 0.00 -> 471.4 mm, vias 0 -> 1
- net ROW2: track 0.00 -> 369.6 mm, vias 0 -> 1
- net ROW1: track 0.00 -> 346.1 mm, vias 0 -> 1
- net COL8: track 0.00 -> 313.5 mm
- net ROW0: track 0.00 -> 307.9 mm, vias 0 -> 1
- net COL0: track 0.00 -> 250.4 mm
- net COL1: track 0.00 -> 229.3 mm
- net COL2: track 0.00 -> 209.0 mm
- net COL3: track 0.00 -> 183.1 mm
- net COL4: track 0.00 -> 178.6 mm
- net COL5: track 0.00 -> 157.7 mm
- net COL6: track 0.00 -> 139.1 mm
- net COL9: track 0.00 -> 114.6 mm
- net COL12: track 0.00 -> 111.1 mm
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Other:
- board size 180 x 277.4 mm -> 388 x 131.2 mm

Commit message: atosukosi
Parts:
- added D70: SOD-123, Diode_SMD:D_SOD-323_HandSoldering, B.Cu at (172.8, 21.5)
- added H1: MountingHole, MountingHole:MountingHole_2.2mm_M2, F.Cu at (26.1, 22.3)
- added H10: MountingHole, MountingHole:MountingHole_2.2mm_M2, F.Cu at (390.2, 22.4)
- added H2: MountingHole, MountingHole:MountingHole_2.2mm_M2, F.Cu at (18.1, 114.3)
- added H3: MountingHole, MountingHole:MountingHole_2.2mm_M2, F.Cu at (170.1, 126.3)
- added H4: MountingHole, MountingHole:MountingHole_2.2mm_M2, F.Cu at (230.2, 41.5)
- added H5: MountingHole, MountingHole:MountingHole_2.2mm_M2, F.Cu at (186.1, 41.3)
- added H6: MountingHole, MountingHole:MountingHole_2.2mm_M2, F.Cu at (107.1, 61.3)
- added H7: MountingHole, MountingHole:MountingHole_2.2mm_M2, F.Cu at (398.2, 114.5)
- added H8: MountingHole, MountingHole:MountingHole_2.2mm_M2, F.Cu at (246.2, 126.5)
- added H9: MountingHole, MountingHole:MountingHole_2.2mm_M2, F.Cu at (309.2, 61.5)
- added J4: HDMI_A_1.4, miyajima:HDMI_A_Sofng_019S, B.Cu at (228.2, 27.8)
- added J5: Conn_01x02, Connector_PinHeader_2.54mm:PinHeader_1x02_P2.54mm_Vertical, F.Cu at (166.9, 21.4)
- J1, USB1: moved to B.Cu
- MX1, MX10, MX11, MX12, MX13, MX14, MX15, MX16, MX18, MX19, MX20, MX21, MX22, MX23, MX24, MX25, MX26, MX27, MX28, MX3, MX30, MX32, MX33, MX34, MX35, MX36, MX37, MX38, MX39, MX4, MX40, MX41, MX42, MX44, MX45, MX49, MX5, MX50, MX53, MX54, MX55, MX56, MX57, MX58, MX6, MX62, MX63, MX67, MX68, MX69, MX7, MX8, MX9: footprint MX_Only:MXOnly-1U-NoLED -> MX_Only:MXOnly-1U-Hotswap
- MX17, MX29: footprint MX_Only:MXOnly-1.75U-NoLED -> MX_Only:MXOnly-1.75U-Hotswap
- MX2: footprint MX_Only:MXOnly-1.5U-NoLED -> MX_Only:MXOnly-1.5U-Hotswap
- MX31, MX43, MX48, MX51: footprint MX_Only:MXOnly-2.25U-ReversedStabilizers-NoLED -> MX_Only:MXOnly-2.25U-Hotswap-ReversedStabilizers
- MX46, MX47, MX52: footprint MX_Only:MXOnly-1.25U-NoLED -> MX_Only:MXOnly-1.25U-Hotswap
- MX59, MX60, MX61, MX64, MX65, MX66: footprint Kailh_Choc:KailhChoc-1U -> miyajima:KailhChoc-1U-hotswap
- SW_BOOT1, SW_RESET1: moved to F.Cu
- moved SW_BOOT1 142.6 mm to (394.2, 105.5), turned to 270 degrees
- moved SW_RESET1 117.1 mm to (394.2, 86.5), turned to 270 degrees
- moved R1 103.9 mm to (242.5, 34.6), turned to 90 degrees
- moved R2 90.1 mm to (268.2, 25.5), turned to 180 degrees
- moved J2 89.1 mm to (269.0, 31.8), turned to 285 degrees
- moved R3 86.4 mm to (276.0, 25.5)
- moved C2 84.9 mm to (249.6, 32.5)
- moved C6 80.3 mm to (253.5, 24.1), turned to 270 degrees
- moved C1 79.2 mm to (254.0, 30.4), turned to 90 degrees
- moved C7 78.9 mm to (245.4, 34.2), turned to 270 degrees
- moved J3 75.3 mm to (278.8, 29.1), turned to 105 degrees
- moved C5 74.9 mm to (246.1, 23.4), turned to 180 degrees
- moved ESD1 56.3 mm to (271.0, 25.6), turned to 180 degrees
- moved ESD2 53.7 mm to (273.2, 25.6), turned to 180 degrees
- moved C3 47.3 mm to (282.0, 22.0), turned to 180 degrees
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Connections:
- J1 pad 1: ROW0 -> ROW4
- J1 pad 10: COL4 -> COL2
- J1 pad 11: COL5 -> COL1
- J1 pad 12: COL6 -> COL0
- J1 pad 2: ROW1 -> ROW3
- J1 pad 4: ROW3 -> ROW1
- J1 pad 5: ROW4 -> ROW0
- J1 pad 6: COL0 -> COL6
- J1 pad 7: COL1 -> COL5
- J1 pad 8: COL2 -> COL4
- U2 pad 1: Net-(U2-Pad1) -> COL8
- U2 pad 10: Net-(U2-Pad10) -> COL4
- U2 pad 11: Net-(U2-Pad11) -> COL5
- U2 pad 12: Net-(U2-Pad12) -> COL6
- U2 pad 13: Net-(U2-Pad13) -> ROW0
- U2 pad 14: Net-(U2-Pad14) -> ROW1
- U2 pad 15: Net-(U2-Pad15) -> ROW2
- U2 pad 18: Net-(U2-Pad18) -> ROW3
- U2 pad 19: Net-(U2-Pad19) -> ROW4
- U2 pad 2: Net-(U2-Pad2) -> COL7
- U2 pad 20: Net-(U2-Pad20) -> COL13
- U2 pad 26: Net-(U2-Pad26) -> COL12
- U2 pad 27: Net-(U2-Pad27) -> COL11
- U2 pad 28: Net-(U2-Pad28) -> COL10
- U2 pad 29: Net-(U2-Pad29) -> COL9
- U2 pad 6: Net-(U2-Pad6) -> COL0
- U2 pad 7: Net-(U2-Pad7) -> COL1
- U2 pad 8: Net-(U2-Pad8) -> COL2
- U2 pad 9: Net-(U2-Pad9) -> COL3
Routing:
- net GND: track 0.00 -> 370.6 mm, vias 0 -> 14
- net +3V3: track 0.00 -> 262.8 mm, vias 0 -> 8
- net Net-(R1-Pad1): track 0.00 -> 258.4 mm, vias 0 -> 5
- net NRST: track 0.00 -> 205.4 mm, vias 0 -> 4
- net ROW3: track 495.5 -> 674.5 mm, vias 1 -> 4
- net ROW4: track 471.4 -> 612.7 mm, vias 1 -> 2
- net COL13: track 109.0 -> 225.1 mm, vias 0 -> 7
- net ROW2: track 369.6 -> 483.6 mm, vias 1 -> 2
- net COL12: track 111.1 -> 203.1 mm, vias 0 -> 5
- net ROW1: track 346.1 -> 432.9 mm, vias 1 -> 2
- net COL11: track 106.1 -> 177.5 mm, vias 0 -> 5
- net COL7: track 107.7 -> 158.7 mm, vias 0 -> 6
- net ROW0: track 307.9 -> 352.5 mm, vias 1 -> 2
- net COL10: track 109.3 -> 152.8 mm, vias 0 -> 6
- net D-: track 0.00 -> 37.6 mm
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- added copper zone on B.Cu, net GND
Other:
- board size 388 x 131.2 mm -> 388 x 126.2 mm
- net class power added: clearance 0.2, trace_width 0.381, via_dia 0.8, via_drill 0.4
- board text added: "3V"
- board text added: "A13"
- board text added: "A14"
- board text added: "C5"
- board text added: "CLK"
- board text added: "DIO"
- board text added: "GND"
- board text added: "OPTSW"
- board text added: "R3"
- board text added: "RST"

Commit message: Dobrock69 kansei!
Parts:
- moved D67 4.07 mm to (330.6, 106.4)
- moved D65 0.66 mm to (292.1, 111.0)
- moved D20 0.20 mm to (121.9, 52.3)
- moved D3 0.20 mm to (79.9, 29.7)
- moved D30 0.20 mm to (41.8, 68.6)
- moved D31 0.20 mm to (46.5, 68.6)
- moved D33 0.20 mm to (106.5, 68.6)
- moved D34 0.20 mm to (126.2, 73.5)
- moved D35 0.20 mm to (144.2, 78.8)
- moved D36 0.20 mm to (162.6, 83.8)
- moved D44 0.20 mm to (45.4, 87.7)
- moved D45 0.20 mm to (66.4, 87.6)
- moved D46 0.20 mm to (88.6, 87.3)
- moved D47 0.20 mm to (96.1, 87.6)
- moved D56 0.20 mm to (45.1, 106.5)
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Routing:
- net ROW3: track 674.5 -> 650.5 mm
- net ROW2: track 483.6 -> 459.9 mm
- net ROW1: track 432.9 -> 411.9 mm
- net GND: track 370.6 -> 352.7 mm
- net COL7: track 158.7 -> 152.3 mm, vias 6 -> 5
- net Net-(R1-Pad1): track 258.4 -> 252.7 mm, vias 5 -> 4
- net COL11: track 177.5 -> 172.8 mm
- net Net-(D67-Pad2): track 25.5 -> 29.6 mm
- net +3V3: track 262.8 -> 266.6 mm
- net COL8: track 331.1 -> 334.9 mm, vias 5 -> 4
- net COL10: track 152.8 -> 149.8 mm
- net ROW4: track 612.7 -> 610.6 mm
- net ROW0: track 352.5 -> 350.5 mm
- net COL13: track 225.1 -> 223.3 mm
- net NRST: track 205.4 -> 203.7 mm
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Other:
- board size 388 x 126.2 mm -> 388 x 126.3 mm
